File: Hardware/calculator copy.kicad_pcb (KiCad board)
At the start: 2 copper layers, 72 x 122 mm, 57 parts, among them J1 Hirose_FH12-28S-0.5SH_1x28-1M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

Commit message: refactor: update PCB component layout and add peripheral utility scripts for hardware maintenance
Parts:
- removed C1, C2, C3, C4, C5, C6, C7, C8: , 
- added C10: C_0402_1005Metric, C_0402_1005Metric, F.Cu at (35.0, -92.0)
- added C11: C_0402_1005Metric, C_0402_1005Metric, F.Cu at (45.0, -96.0)
- added C12: C_0402_1005Metric, C_0402_1005Metric, F.Cu at (55.0, -92.0)
- moved J1 3.00 mm to (45.0, -92.0)
Connections:
- J1 pad 1: (no net) -> Net-(J1-Pad1)
- J1 pad 10: (no net) -> Net-(J1-Pad10)
- J1 pad 13: Net-(J1-Pad13) -> (no net)
- J1 pad 14: Net-(J1-Pad14) -> (no net)
- J1 pad 15: +3V3 -> (no net)
- J1 pad 16: GND -> (no net)
- J1 pad 17: Net-(J1-Pad17) -> (no net)
- J1 pad 18: Net-(J1-Pad18) -> (no net)
- J1 pad 19: Net-(J1-Pad19) -> (no net)
- J1 pad 20: Net-(J1-Pad20) -> (no net)
- J1 pad 21: Net-(J1-Pad21) -> (no net)
- J1 pad 22: Net-(J1-Pad22) -> (no net)
- J1 pad 23: Net-(J1-Pad23) -> (no net)
- J1 pad 24: Net-(J1-Pad24) -> (no net)
- J1 pad 25: Net-(J1-Pad25) -> (no net)
- J1 pad 26: Net-(J1-Pad26) -> (no net)
- J1 pad 27: GND -> (no net)
- J1 pad 28: GND -> (no net)
- J1 pad 5: GND -> Net-(J1-Pad5)
- J1 pad 6: GND -> +3V3
- J1 pad 7: (no net) -> GND
- J1 pad 8: (no net) -> Net-(J1-Pad8)
- J1 pad 9: (no net) -> Net-(J1-Pad9)
Other:
- board size 72 x 122 mm -> 72 x 138 mm
