File: Hardware/temp.kicad_pcb (KiCad board)
At the start: 2 copper layers, 72 x 122 mm, 57 parts, among them J1 Hirose_FH12-28S-0.5SH_1x28-1M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

Commit message: refactor: update PCB component layout and add peripheral utility scripts for hardware maintenance
Parts:
- removed C1, C2, C3, C4, C5, C6, C7, C8: , 
- added C10: C_0402_1005Metric, C_0402_1005Metric, F.Cu at (35.0, -99.0)
- added C11: C_0402_1005Metric, C_0402_1005Metric, F.Cu at (37.5, -99.0)
- added C12: C_0402_1005Metric, C_0402_1005Metric, F.Cu at (40.0, -99.0)
- added C13: C_0402_1005Metric, C_0402_1005Metric, F.Cu at (42.5, -99.0)
- added C14: C_0402_1005Metric, C_0402_1005Metric, F.Cu at (45.0, -99.0)
- added C15: C_0402_1005Metric, C_0402_1005Metric, F.Cu at (47.5, -99.0)
- added C16: C_0402_1005Metric, C_0402_1005Metric, F.Cu at (50.0, -99.0)
- added C17: C_0402_1005Metric, C_0402_1005Metric, F.Cu at (52.5, -99.0)
