File: Hardware/calculator.kicad_pcb (KiCad board)
At the start: 2 copper layers, 72 x 122 mm, 57 parts, among them J1 Hirose_FH12-28S-0.5SH_1x28-1M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

Commit message: refactor: add watchOS slider UI, update PCB hardware layouts, and enable fraction entry testing
Parts:
- removed FID1, FID2, FID3: Fiducial_1mm_Mask2mm, Fiducial:Fiducial_1mm_Mask2mm
- C1, C2, C3, C4, C5, C6, C7, C8: moved to B.Cu
- J1: value Hirose_FH12-28S-0.5SH_1x28-1MP_P0.50mm_Horizontal -> (none); footprint Hirose_FH12-28S-0.5SH_1x28-1MP_P0.50mm_Horizontal -> (none)
- moved C1 13.1 mm to (36.2, -93.0), turned to 180 degrees
- moved C2 13.1 mm to (38.8, -93.0), turned to 180 degrees
- moved C3 13.1 mm to (41.2, -93.0), turned to 180 degrees
- moved C4 13.1 mm to (43.8, -93.0), turned to 180 degrees
- moved C5 13.1 mm to (46.2, -93.0), turned to 180 degrees
- moved C6 13.1 mm to (48.8, -93.0), turned to 180 degrees
- moved C7 13.1 mm to (51.2, -93.0), turned to 180 degrees
- moved C8 13.1 mm to (53.8, -93.0), turned to 180 degrees
- moved B21 9.10 mm to (16.2, -2.90)
- moved B25 9.10 mm to (32.7, -2.90)
- moved B29 9.10 mm to (46.4, -2.90)
- moved B33 9.10 mm to (60.1, -2.90)
- moved B37 9.10 mm to (73.8, -2.90)
- moved B20 7.80 mm to (16.2, -14.2)
- moved B24 7.80 mm to (32.7, -14.2)
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Connections:
- J1 pad 13: Net-(J1-Pad13) -> SPI_SCK
- J1 pad 14: Net-(J1-Pad14) -> SPI_MOSI
- J1 pad 15: +3V3 -> (no net)
- J1 pad 16: GND -> (no net)
- J1 pad 17: Net-(J1-Pad17) -> (no net)
- J1 pad 18: Net-(J1-Pad18) -> (no net)
- J1 pad 19: Net-(J1-Pad19) -> (no net)
- J1 pad 2: Net-(J1-Pad2) -> SPI_CS
- J1 pad 20: Net-(J1-Pad20) -> (no net)
- J1 pad 21: Net-(J1-Pad21) -> (no net)
- J1 pad 22: Net-(J1-Pad22) -> (no net)
- J1 pad 23: Net-(J1-Pad23) -> (no net)
- J1 pad 24: Net-(J1-Pad24) -> (no net)
- J1 pad 25: Net-(J1-Pad25) -> (no net)
- J1 pad 26: Net-(J1-Pad26) -> (no net)
- J1 pad 27: GND -> (no net)
- J1 pad 28: GND -> (no net)
- J1 pad 3: Net-(J1-Pad3) -> RST
- J1 pad 4: Net-(J1-Pad4) -> SPI_DC
- J1 pad 5: GND -> (no net)
- J1 pad 6: GND -> (no net)
- MCU1 pad 10: P14 -> P7
- MCU1 pad 11: P16 -> P8
- MCU1 pad 12: P10 -> P9
- MCU1 pad 13: P1 -> SPI_CS
- MCU1 pad 14: P0 -> P10
- MCU1 pad 17: P2 -> SPI_SCK
- MCU1 pad 18: GND -> SPI_MOSI
- MCU1 pad 19: P4 -> SPI_DC
- MCU1 pad 20: P5 -> P14
- MCU1 pad 21: P6 -> P15
- MCU1 pad 22: Net-(J1-Pad1) -> P16
- MCU1 pad 23: GND -> P20
- MCU1 pad 24: Net-(J1-Pad4) -> P21
- MCU1 pad 5: P21 -> P0
- MCU1 pad 6: P20 -> P1
- MCU1 pad 7: P19 -> P4
- MCU1 pad 8: P18 -> P5
- MCU1 pad 9: P15 -> P6
Routing:
- net GND: track 206.6 -> 1198.4 mm, vias 1 -> 11
- net P10: track 294.8 -> 759.2 mm, vias 4 -> 5
- net P19: track 0.00 -> 371.2 mm, vias 0 -> 1
- net P20: track 217.2 -> 453.9 mm
- net P5: track 338.7 -> 563.8 mm, vias 4 -> 6
- net P0: track 278.0 -> 492.5 mm
- net P21: track 364.1 -> 195.6 mm
- net P1: track 298.8 -> 145.9 mm, vias 4 -> 5
- net P6: track 286.7 -> 436.9 mm, vias 6 -> 7
- net P15: track 264.8 -> 411.1 mm
- net P14: track 264.5 -> 408.1 mm
- net P16: track 164.7 -> 294.0 mm
- net P4: track 230.6 -> 118.2 mm, vias 4 -> 5
- net P9: track 168.0 -> 259.9 mm
- net P7: track 168.4 -> 76.7 mm
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Other:
- board size 72 x 122 mm -> 72 x 142.4 mm

Commit message: Fix WatchOS UI lockups, STO+ UX, REGS/VIEW features, and SIG mode auto-tracking math
Parts:
- MCU1: value RASPBERRY PI PICO -> (none); footprint ProMicro -> (none)
- moved MCU1 13.1 mm to (21.5, -102.5), turned to 0 degrees
Connections:
- J1 pad 3: RST -> SPI_RES
- MCU1 pad 1: RAW -> (no net)
- MCU1 pad 10: P7 -> P1
- MCU1 pad 11: P8 -> P4
- MCU1 pad 12: P9 -> P5
- MCU1 pad 13: SPI_CS -> GND
- MCU1 pad 14: P10 -> P6
- MCU1 pad 15: GND -> P7
- MCU1 pad 16: GND -> P8
- MCU1 pad 17: SPI_SCK -> P9
- MCU1 pad 18: SPI_MOSI -> GND
- MCU1 pad 19: SPI_DC -> P10
- MCU1 pad 2: GND -> SPI_CS
- MCU1 pad 23: P20 -> GND
- MCU1 pad 24: P21 -> P20
- MCU1 pad 3: RST -> GND
- MCU1 pad 4: VCC -> SPI_SCK
- MCU1 pad 5: P0 -> SPI_MOSI
- MCU1 pad 6: P1 -> SPI_DC
- MCU1 pad 7: P4 -> SPI_RES
- MCU1 pad 8: P5 -> GND
- MCU1 pad 9: P6 -> P0
Routing:
- net GND: track 1198.4 -> 2102.4 mm
- net P10: track 759.2 -> 1283.6 mm
- net P5: track 563.8 -> 1045.8 mm, vias 6 -> 7
- net P14: track 408.1 -> 850.8 mm, vias 1 -> 3
- net P20: track 453.9 -> 887.0 mm, vias 1 -> 2
- net P15: track 411.1 -> 800.1 mm, vias 1 -> 2
- net P6: track 436.9 -> 818.5 mm, vias 7 -> 9
- net P0: track 492.5 -> 832.6 mm
- net P9: track 259.9 -> 537.4 mm, vias 0 -> 2
- net P8: track 251.8 -> 491.2 mm, vias 0 -> 2
- net P16: track 294.0 -> 522.4 mm
- net P21: track 195.6 -> 392.8 mm
- net P1: track 145.9 -> 292.8 mm
- net P4: track 118.2 -> 249.1 mm, vias 5 -> 6
- net P7: track 76.7 -> 189.8 mm, vias 0 -> 1
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